Commit message: Add SDF demo descripton.

File: demo_common/demo_description/robots/demo_model.urdf.xacro (robot description, xacro)
@@ -5,5 +5,5 @@
   <link name="base_link"/>
   <xacro:stick parent="base_link" suffix="A">
-    <origin xyz="0 0 0" rpy="${M_PI/2} 0 ${M_PI/2}"/>
+    <origin xyz="0 0 0" rpy="0 0 0"/>
   </xacro:stick>
   <xacro:stick parent="stick_A" suffix="B">

File: demo_common/demo_description/urdf/stick.urdf.xacro (robot description, xacro)
@@ -17,5 +17,5 @@
     </link>
     <joint name="${parent}_to_stick_${suffix}" type="continuous">
-      <axis xyz="0 0 1"/>
+      <axis xyz="0 1 0"/>
       <parent link="${parent}"/>
       <child link="stick_${suffix}"/>

Commit message: fix description

File: demo_common/demo_description/robots/demo_model.urdf.xacro (robot description, xacro)
@@ -4,5 +4,5 @@
   <xacro:include filename="$(find demo_description)/urdf/closed_link.urdf.xacro"/>
   <link name="base_link"/>
-  <xacro:closed_link parent="base_link" suffix="A">
+  <xacro:closed_link parent="base_link">
     <origin xyz="0 0 0" rpy="0 0 ${M_PI/4}"/>
   </xacro:closed_link>

File: demo_common/demo_description/urdf/closed_link.urdf.xacro (robot description, xacro)
@@ -3,5 +3,5 @@
   <xacro:include filename="$(find demo_description)/urdf/common.xacro"/>
   <xacro:include filename="$(find demo_description)/urdf/closed_link.transmission.xacro"/>
-  <xacro:macro name="closed_link" params="parent suffix *joint_origin">
+  <xacro:macro name="closed_link" params="parent *joint_origin">
     <link name="link_A">
       <visual>
