Commit message: Change the structure of the model.

File: demo_common/demo_description/robots/demo_model.urdf (robot description, URDF)
Before this commit: robot demo_model, 5 links, 4 joints
Links:
- removed link stick_A
- removed link stick_B
- removed link stick_C
- removed link stick_D
- added link link_A; collision box size=2. 0.1 0.1; visual box size=2.0 0.1 0.1
- added link link_B; collision box size=2. 0.1 0.1; visual box size=2.0 0.1 0.1
- added link link_C; collision box size=2. 0.1 0.1; visual box size=2.0 0.1 0.1
- added link link_D; collision box size=2. 0.1 0.1; visual box size=2.0 0.1 0.1
Joints:
- removed joint base_link_to_stick_A
- removed joint stick_A_to_stick_B
- removed joint stick_B_to_stick_C
- removed joint stick_C_to_stick_D
- added joint base_link_to_link_A: type revolute, parent base_link, child link_A, origin xyz=0 0 0 rpy=0 0 0.785398185, axis 0 0 1, limit lower=-0.785398185 upper=0.785398185 effort=100.0 velocity=3.14159274
- added joint link_A_to_link_B: type continuous, parent link_A, child link_B, origin xyz=2 0 0 rpy=0 0 -1.57079637, axis 0 0 1
- added joint link_B_to_link_C: type continuous, parent link_B, child link_C, origin xyz=2 0 0 rpy=0 0 -1.57079637, axis 0 0 1
- added joint link_C_to_link_D: type continuous, parent link_C, child link_D, origin xyz=2 0 0 rpy=0 0 -1.57079637, axis 0 0 1

File: demo_common/demo_description/robots/demo_model.urdf.xacro (robot description, xacro)
@@ -2,17 +2,8 @@
 <robot name="demo_model" xmlns:xacro="http://ros.org/wiki/xacro">
   <xacro:include filename="$(find demo_description)/urdf/common.xacro"/>
-  <xacro:include filename="$(find demo_description)/urdf/stick.urdf.xacro"/>
+  <xacro:include filename="$(find demo_description)/urdf/closed_link.urdf.xacro"/>
   <link name="base_link"/>
-  <xacro:stick parent="base_link" suffix="A">
-    <origin xyz="0 0 0" rpy="0 0 0"/>
-  </xacro:stick>
-  <xacro:stick parent="stick_A" suffix="B">
-    <origin xyz="2 0 0" rpy="0 0 0"/>
-  </xacro:stick>
-  <xacro:stick parent="stick_B" suffix="C">
-    <origin xyz="2 0 0" rpy="0 0 0"/>
-  </xacro:stick>
-  <xacro:stick parent="stick_C" suffix="D">
-    <origin xyz="2 0 0" rpy="0 0 0"/>
-  </xacro:stick>
+  <xacro:closed_link parent="base_link" suffix="A">
+    <origin xyz="0 0 0" rpy="0 0 ${M_PI/4}"/>
+  </xacro:closed_link>
 </robot>

Commit message: Fix effort controller

File: demo_common/demo_description/robots/demo_model.urdf (robot description, URDF)
Before this commit: robot demo_model, 5 links, 4 joints
Joints:
- joint base_link_to_link_A: axis 0 0 1 -> (none); limit lower=-0.785398185 upper=0.785398185 effort=100.0 velocity=3.14159274 -> (none); type revolute -> fixed
- joint link_A_to_link_B: limit (none) -> lower=-0.785398185 upper=0.785398185 effort=100.0 velocity=3.14159274; type continuous -> revolute

File: demo_common/demo_description/robots/demo_model.urdf.xacro (robot description, xacro)
@@ -5,5 +5,5 @@
   <link name="base_link"/>
   <xacro:closed_link parent="base_link">
-    <origin xyz="0 0 0" rpy="0 0 ${M_PI/4}"/>
+    <origin xyz="0 0 0" rpy="0 0 0"/>
   </xacro:closed_link>
 </robot>

File: demo_common/demo_description/urdf/closed_link.urdf.xacro (robot description, xacro)
@@ -60,19 +60,18 @@
       </collision>
     </link>
-    <joint name="${parent}_to_link_A" type="revolute">
-      <axis xyz="0 0 1"/>
-      <limit lower="${-M_PI/4}" upper="${M_PI/4}" effort="100.0" velocity="${M_PI}"/>
-      <dynamics damping="0.1"/>
+    <joint name="${parent}_to_link_A" type="fixed">
       <parent link="${parent}"/>
       <child link="link_A"/>
       <xacro:insert_block name="joint_origin"/>
     </joint>
-    <xacro:effort_trans joint="${parent}_to_link_A"/>
-    <joint name="link_A_to_link_B" type="continuous">
+    <joint name="link_A_to_link_B" type="revolute">
       <axis xyz="0 0 1"/>
+      <limit lower="${-M_PI/4}" upper="${M_PI/4}" effort="100.0" velocity="${M_PI}"/>
+      <dynamics damping="0.1"/>
       <parent link="link_A"/>
       <child link="link_B"/>
       <origin xyz="2 0 0" rpy="0 0 ${-M_PI/2}"/>
     </joint>
+    <xacro:effort_trans joint="link_A_to_link_B"/>
     <joint name="link_B_to_link_C" type="continuous">
       <axis xyz="0 0 1"/>
